File: FDC_2214_Breakout/FDC_2214_Breakout.kicad_pcb (KiCad board)
At the start: 2 copper layers, 32.7 x 32.7 mm, 51 parts, among them J1 Sensor_2, J2 Sensor_1, J3 Sensor_0, J4 Sensor_3, J5 I/O, U1 FDC2214RGHT, U2 625L3C040M00000

Commit message: Kicad Export
Parts:
- added G***: LOGO, qr_code:qr_FDC, F.Cu at (171.3, 108.1)
- moved C4 13.2 mm to (191.4, 124.7), turned to 90 degrees
- moved C22 6.65 mm to (191.4, 114.8)
- moved C18 5.99 mm to (191.4, 108.0), turned to 90 degrees
- moved C17 5.93 mm to (173.6, 113.0), turned to 180 degrees
- moved C16 5.57 mm to (182.6, 111.0), turned to 180 degrees
- moved C20 4.83 mm to (191.4, 121.5)
- moved C1 4.45 mm to (186.0, 120.5)
- moved C10 3.89 mm to (181.4, 128.0)
- moved C5 3.41 mm to (176.6, 118.6)
- moved C23 2.96 mm to (191.4, 111.3)
- moved C12 2.52 mm to (170.7, 119.7)
- moved C13 2.07 mm to (173.6, 115.0)
- moved C15 2.02 mm to (185.9, 112.9)
- moved C21 1.50 mm to (191.4, 118.2)
- moved C9 0.58 mm to (178.0, 128.0)
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Routing:
- net In2B: track 9.65 -> 20.8 mm
- net Net-(J2-Pin_2): track 12.3 -> 20.7 mm
- net Net-(J2-Pin_1): track 11.1 -> 18.7 mm
- net In1B: track 6.18 -> 12.2 mm
- net In0A: track 6.52 -> 11.5 mm
- net In3B: track 6.77 -> 10.6 mm
- net Net-(J3-Pin_2): track 12.7 -> 16.3 mm
- net In2A: track 5.89 -> 9.40 mm
- net In3A: track 12.2 -> 15.5 mm
- net In0B: track 12.1 -> 14.8 mm
- net Net-(J4-Pin_1): track 11.8 -> 14.2 mm
- net In1A: track 10.5 -> 12.7 mm
- net Net-(J1-Pin_1): track 14.6 -> 12.4 mm
- net Net-(J3-Pin_1): track 11.2 -> 12.6 mm
- net Net-(J4-Pin_2): track 15.8 -> 15.0 mm
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Other:
- board text removed: "QR CODE TO GITHUB HERE"
